Commit message: mobile manipulator mpc

File: ocs2_robotic_assets/resources/mobile_manipulator/franka/urdf/panda.urdf (robot description, URDF)
Before this commit: robot panda, 14 links, 13 joints
Links:
- removed link panda_hand
- removed link panda_hand_tcp
- removed link panda_leftfinger
- removed link panda_link0
- removed link panda_link1
- removed link panda_link2
- removed link panda_link3
- removed link panda_link4
- removed link panda_link5
- removed link panda_link6
- removed link panda_link7
- removed link panda_link8
- removed link panda_rightfinger
- removed link root
- added link panda
- added link panda_panda_hand; collision mesh filename=package://ocs2_robotic_assets/resources/mobile_manipulator/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 scale=1. 1. 1.; visual mesh filename=package://ocs2_robotic_assets/resources/mobile_manipulator/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 scale=0.01 0.01 0.01
- added link panda_panda_leftfinger; collision mesh filename=package://ocs2_robotic_assets/resources/mobile_manipulator/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 scale=1. 1. 1.; visual mesh filename=package://ocs2_robotic_assets/resources/mobile_manipulator/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 scale=0.01 0.01 0.01
- added link panda_panda_link0; collision mesh filename=package://ocs2_robotic_assets/resources/mobile_manipulator/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 scale=1. 1. 1.; visual mesh filename=package://ocs2_robotic_assets/resources/mobile_manipulator/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 scale=0.01 0.01 0.01
- added link panda_panda_link1; collision mesh filename=package://ocs2_robotic_assets/resources/mobile_manipulator/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 scale=1. 1. 1.; visual mesh filename=package://ocs2_robotic_assets/resources/mobile_manipulator/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 scale=0.01 0.01 0.01
- added link panda_panda_link2; collision mesh filename=package://ocs2_robotic_assets/resources/mobile_manipulator/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 scale=1. 1. 1.; visual mesh filename=package://ocs2_robotic_assets/resources/mobile_manipulator/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 scale=0.01 0.01 0.01
- added link panda_panda_link3; collision mesh filename=package://ocs2_robotic_assets/resources/mobile_manipulator/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 scale=1. 1. 1.; visual mesh filename=package://ocs2_robotic_assets/resources/mobile_manipulator/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 scale=0.01 0.01 0.01
- added link panda_panda_link4; collision mesh filename=package://ocs2_robotic_assets/resources/mobile_manipulator/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 scale=1. 1. 1.; visual mesh filename=package://ocs2_robotic_assets/resources/mobile_manipulator/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 scale=0.01 0.01 0.01
- added link panda_panda_link5; collision mesh filename=package://ocs2_robotic_assets/resources/mobile_manipulator/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 scale=1. 1. 1.; visual mesh filename=package://ocs2_robotic_assets/resources/mobile_manipulator/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 scale=0.01 0.01 0.01
- added link panda_panda_link6; collision mesh filename=package://ocs2_robotic_assets/resources/mobile_manipulator/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 scale=1. 1. 1.; visual mesh filename=package://ocs2_robotic_assets/resources/mobile_manipulator/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 scale=0.01 0.01 0.01
- added link panda_panda_link7; collision mesh filename=package://ocs2_robotic_assets/resources/mobile_manipulator/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 scale=1. 1. 1.; visual mesh filename=package://ocs2_robotic_assets/resources/mobile_manipulator/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 scale=0.01 0.01 0.01
- added link panda_panda_rightfinger; collision mesh filename=package://ocs2_robotic_assets/resources/mobile_manipulator/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 scale=1. 1. 1.; visual mesh filename=package://ocs2_robotic_assets/resources/mobile_manipulator/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 scale=0.01 0.01 0.01
Joints:
- removed joint panda_hand_tcp_joint
- removed joint panda_joint8
- removed joint root_joint
- added joint rootJoint: type fixed, parent panda, child panda_panda_link0, origin xyz=0. 0. 0. rpy=0. 0. 0.
- joint panda_finger_joint1: axis 0 1 0 -> 1. 0. 0.; child panda_leftfinger -> panda_panda_leftfinger; limit lower=0.0 upper=0.04 effort=100 velocity=0.2 -> lower=0. upper=0.04 effort=200. velocity=0.2; origin xyz=0 0 0.0584 rpy=0 0 0 -> xyz=0. 0. 0.0584 rpy=0. 0. 1.5707964; parent panda_hand -> panda_panda_hand
- joint panda_finger_joint2: axis 0 -1 0 -> 1. 0. 0.; child panda_rightfinger -> panda_panda_rightfinger; limit lower=0.0 upper=0.04 effort=100 velocity=0.2 -> lower=0. upper=0.04 effort=200. velocity=0.2; mimic joint=panda_finger_joint1 -> (none); origin xyz=0 0 0.0584 rpy=0 0 0 -> xyz=0. 0. 0.0584 rpy=0. 0. -1.5707964; parent panda_hand -> panda_panda_hand
- joint panda_hand_joint: child panda_hand -> panda_panda_hand; origin xyz=0 0 0 rpy=0 0 -0.7853981633974483 -> xyz=0.107 0. 0.  rpy=-1.5707964 0.7853981 -1.5707964; parent panda_link8 -> panda_panda_link7
- joint panda_joint1: axis 0 0 1 -> 1. 0. 0.; child panda_link1 -> panda_panda_link1; limit lower=-2.8973 upper=2.8973 effort=87 velocity=2.1750 -> lower=-2.8973001 upper=2.8973001 effort=87. velocity=2.1749999; origin xyz=0 0 0.333 rpy=0 0 0 -> xyz=0. 0. 0.333 rpy=0. -1.5707963 0. ; parent panda_link0 -> panda_panda_link0
- joint panda_joint2: axis 0 0 1 -> 1. 0. 0.; child panda_link2 -> panda_panda_link2; limit lower=-1.7628 upper=1.7628 effort=87 velocity=2.1750 -> lower=-1.7628 upper=1.7628 effort=87. velocity=2.1749999; origin xyz=0 0 0 rpy=-1.5707963267948966 0 0 -> xyz=0. 0. 0. rpy=0. 0. 1.5707964; parent panda_link1 -> panda_panda_link1
- joint panda_joint3: axis 0 0 1 -> 1. 0. 0.; child panda_link3 -> panda_panda_link3; limit lower=-2.8973 upper=2.8973 effort=87 velocity=2.1750 -> lower=-2.8973001 upper=2.8973001 effort=87. velocity=2.1749999; origin xyz=0 -0.316 0 rpy=1.5707963267948966 0 0 -> xyz=0. -0.316 0.  rpy=0. 0. -1.5707964; parent panda_link2 -> panda_panda_link2
- joint panda_joint4: axis 0 0 1 -> 1. 0. 0.; child panda_link4 -> panda_panda_link4; limit lower=-3.0718 upper=-0.0698 effort=87 velocity=2.1750 -> lower=-3.0718 upper=-0.0698 effort=87. velocity=2.1749999; origin xyz=0.0825 0 0 rpy=1.5707963267948966 0 0 -> xyz=0. 0. -0.0825 rpy=0. 0. -1.5707964; parent panda_link3 -> panda_panda_link3
- joint panda_joint5: axis 0 0 1 -> 1. 0. 0.; child panda_link5 -> panda_panda_link5; limit lower=-2.8973 upper=2.8973 effort=12 velocity=2.6100 -> lower=-2.8973001 upper=2.8973001 effort=12. velocity=2.6100004; origin xyz=-0.0825 0.384 0 rpy=-1.5707963267948966 0 0 -> xyz=0. 0.384 0.0825 rpy=0. 0. 1.5707964; parent panda_link4 -> panda_panda_link4
- joint panda_joint6: axis 0 0 1 -> 1. 0. 0.; child panda_link6 -> panda_panda_link6; limit lower=-0.0175 upper=3.7525 effort=12 velocity=2.6100 -> lower=-0.0175 upper=3.7525 effort=12. velocity=2.6100004; origin xyz=0 0 0 rpy=1.5707963267948966 0 0 -> xyz=0. 0. 0. rpy=0. 0. -1.5707964; parent panda_link5 -> panda_panda_link5
- joint panda_joint7: axis 0 0 1 -> 1. 0. 0.; child panda_link7 -> panda_panda_link7; limit lower=-2.8973 upper=2.8973 effort=12 velocity=2.6100 -> lower=-2.8973001 upper=2.8973001 effort=12. velocity=2.6100004; origin xyz=0.088 0 0 rpy=1.5707963267948966 0 0 -> xyz=0. 0. -0.088 rpy=0. 0. -1.5707964; parent panda_link6 -> panda_panda_link6
