Commit message: kinova

File: ocs2_robotic_assets/resources/mobile_manipulator/kinova/urdf/j2n6s300.urdf (robot description, URDF)
Before this commit: robot j2n6s300, 15 links, 14 joints
Links:
- removed link j2n6s300_link_finger_1
- removed link j2n6s300_link_finger_2
- removed link j2n6s300_link_finger_3
- removed link j2n6s300_link_finger_tip_1
- removed link j2n6s300_link_finger_tip_2
- removed link j2n6s300_link_finger_tip_3
Joints:
- removed joint j2n6s300_joint_finger_1
- removed joint j2n6s300_joint_finger_2
- removed joint j2n6s300_joint_finger_3
- removed joint j2n6s300_joint_finger_tip_1
- removed joint j2n6s300_joint_finger_tip_2
- removed joint j2n6s300_joint_finger_tip_3
