Commit message: relative

File: ocs2_robotic_assets/resources/mobile_manipulator/stick/urdf/stick.urdf (robot description, URDF)
Before this commit: robot stick, 2 links, 1 joints
Joints:
- joint interaction_joint: limit lower=-1000 upper=1000 effort=100 velocity=100 -> lower=0 upper=0 effort=0 velocity=0; origin xyz=0 0 0 rpy=0 0 0 -> xyz=0.1 -0.8 0 rpy=0 0 0

Commit message: push

File: ocs2_robotic_assets/resources/mobile_manipulator/stick/urdf/stick.urdf (robot description, URDF)
Before this commit: robot stick_, 2 links, 1 joints
Joints:
- joint interaction_joint: origin xyz=0.1 -0.8 0 rpy=0 0 0 -> xyz=0 -0.6 0.1 rpy=0 0 0

Commit message: push2

File: ocs2_robotic_assets/resources/mobile_manipulator/stick/urdf/stick.urdf (robot description, URDF)
Before this commit: robot stick_, 2 links, 1 joints
Joints:
- joint interaction_joint: origin xyz=0 -0.6 0.1 rpy=0 0 0 -> xyz=0.8 0.0 0.1 rpy=0 0 0
